File: EvoBorne_pcb/evoborne_pcb/evoborne.kicad_pcb (KiCad board)
At the start: 2 copper layers, 80.9 x 92.7 mm, 124 parts, among them J1 B2B-XH-A_LF__SN_, J10 XT60, J11 Conn_01x08_Male, J12 Conn_01x08_Male, J13 Screw_Terminal_01x02, J14 USB_C_Receptacle_USB2.0, J15 Conn_01x08_Male, J16 Conn_01x14_Pin, J17 Conn_01x14_Pin, J18 Conn_01x02_Pin, J19 Conn_01x02_Pin, J2 B2B-XH-A_LF__SN_, J3 B2B-XH-A_LF__SN_, J4 B2B-XH-A_LF__SN_, J5 Conn_01x03_Pin, J6 Conn_01x03_Pin, J7 Conn_01x03_Pin, J8 Conn_01x03_Pin, J9 XT60, Q1 SS8050, Q2 SS8050, SW2 SW_N20, SW3 SW_Servos, SW4 SW_Jetson, SW5 EN, SW6 BOOT, SW7_4 SW_Push_Dual, SW8_2 SW_Push_Dual, U1 TB6612FNG, U2 AMS1117, U3 ESP32-WROOM Chip, U4 XL4015, U5 XL4015, U6 XL4015, U7 CH340G, Y1 12MHz

Commit message: PCB files updated
Parts:
- removed the G*** at (73.9, 78.2)
- removed the G*** at (112.5, 78.0)
- added F3: 300mA, PTC Fuse:1A PTC Fuse RXEF050, F.Cu at (69.5, 145.5)
- added G***: LOGO, Logos:Lions Circuit Footprint, B.Cu at (76.5, 142.5)
- added G***: LOGO, Logos:SRA Footprint, B.Cu at (75.5, 128.6)
- added G***: LOGO, Logos:EvoBorne Footprint, B.Cu at (74.2, 77.9)
- C21: value 22pF -> 22 pF
- C22: value 0.1uF -> 0.1 uF
- C23: value 0.1 uF -> 0.1uF
- C5: value +220uF -> 220uF
- D10: renamed from +D10; value 13 -> LED
- D11: renamed from +D11; value 25 -> LED
- D12: renamed from D12+; value 26 -> LED
- D13: renamed from D13+; value 5 -> LED
- D14: renamed from D14+; value 15 -> LED
- D15: renamed from D15+; value 18 -> LED
- D16: renamed from D16+; value 19 -> LED
- D17: renamed from D17+; value 8.4V -> LED
- D18: value 3V3+ -> LED
- D19: renamed from D19+; value 12V -> LED
- D2: renamed from +D2; value 24V -> LED
- D20: renamed from D20+; value 24V_ESC -> LED
- D5: renamed from D5+; value 5V -> LED
- D9: renamed from +D9; value 12 -> LED
- R29: renamed from R29,28; value 5.1 -> 5.1k
- R5: value 24V-12V -> TrimPOT 3296
- R6: value 24V-8.4V -> TrimPOT 3296
- R7: value 24V-5V -> TrimPOT 3296
- SW1: renamed from SW_1; value SW_ESC -> High Current 3 Pin spdt Switch
- U2: value AMS1117 -> AMS1117-3.3
- moved G*** 58.8 mm to (121.5, 103.0)
- moved J18 0.78 mm to (72.1, 111.0)
- moved R24 0.55 mm to (127.8, 129.6)
- moved D20 0.43 mm to (127.8, 127.8)
- moved C18 0.21 mm to (123.2, 81.1)
- renumbered C11+ to C11, C19+ to C19, +C9 to C9, SW7_4 to SW7, SW8_2 to SW8
Connections:
- R10 pad 2: /3V3 -> /3V3_P
Routing:
- net /3V3_P: track 0.00 -> 101.5 mm, vias 0 -> 3
- net /3V3: track 131.2 -> 200.7 mm, vias 1 -> 5
- net GND: track 72.0 -> 94.6 mm, vias 2 -> 5
- net (no net): track 11.3 -> 22.4 mm
- net /24V: track 221.4 -> 228.7 mm
- net /23: track 99.9 -> 104.1 mm
- net Net-(D3-K): track 18.3 -> 20.9 mm
- net /TXD: track 43.6 -> 45.5 mm
- net Net-(D8-K): track 18.8 -> 20.3 mm
- net Net-(U6-VC): track 38.9 -> 37.8 mm
- net Net-(U6-FB): track 136.5 -> 137.2 mm
- net Net-(U7-XO): track 15.3 -> 16.0 mm
Other:
- board text added: "0"
- board text added: "12"
- board text added: "12V"
- board text added: "13"
- board text added: "14"
- board text added: "15"
- board text added: "16"
- board text added: "17"
- board text added: "18"
- board text added: "19"
- board text added: "2"
- board text added: "21"
- board text added: "22"
- board text added: "23"
- board text added: "25"
- board text added: "26"
- board text added: "27"
- board text added: "32"
- board text added: "33"
- board text added: "34"
- board text added: "35"
- board text added: "3V3"
- board text added: "4"
- board text added: "5"
- board text added: "A1"
- board text added: "A2"
- board text added: "B1"
- board text added: "B2"
- board text added: "EN"
- board text added: "GND"
- board text added: "M1A"
- board text added: "M1B"
- board text added: "M2A"
- board text added: "M2B"
- board text added: "VN"
- board text added: "VP"
