File: EvoBorne_pcb/evoborne_pcb/evoborne.kicad_sch (KiCad schematic)
At the start: 121 parts, among them J1 B2B-XH-A_LF__SN_, J10 XT60, J11 Conn_01x08_Male, J12 Conn_01x08_Male, J13 Screw_Terminal_01x02, J15 Conn_01x08_Male, J16 Conn_01x14_Pin, J17 Conn_01x14_Pin, J18 Conn_01x02_Pin, J19 Conn_01x02_Pin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

Commit message: PCB files updated
Parts:
- added F3: 300mA, PTC Fuse:1A PTC Fuse RXEF050, symbol Device:Fuse
Connections:
- net 3V3: now also F3.1; no longer R10.2
- new net 3V3_P: F3.2, R10.2
